Commit message: vorige urdf

File: description/robot.urdf.xacro (robot description, xacro)
@@ -1,4 +1,11 @@
 <?xml version="1.0"?>
 <robot xmlns:xacro="http://www.ros.org/wiki/xacro"  name="robot">
+    <xacro:if value="$(arg use_ros2_control)">
+        <xacro:include filename="ros2_control.xacro" />
+    </xacro:if>
+    <xacro:unless value="$(arg use_ros2_control)">
+        <xacro:include filename="gazebo_control.xacro" />
+    </xacro:unless>
     <xacro:include filename="robot_core.xacro" />
+    <xacro:include filename="lidar.xacro" />
 </robot>

File: description/robot_core.xacro (robot description, xacro)
@@ -44,4 +44,7 @@
         </xacro:inertial_box>
     </link>
+    <gazebo reference="chassis">
+        <material>Gazebo/Red</material>
+    </gazebo>
     <!--  LEFT WHEEL LINK  -->
     <joint name="left_wheel_joint" type="continuous">
@@ -60,5 +63,5 @@
         <collision>
             <geometry>
-                <cylinder length="0.08" radius="0.17" />/>
+                <sphere radius="0.17" />/>
             </geometry>
         </collision>
@@ -67,4 +70,7 @@
         </xacro:inertial_cylinder>
     </link>
+    <gazebo reference="left_wheel">
+        <material>Gazebo/Grey</material>
+    </gazebo>
     <!-- RIGHT WHEEL -->
     <joint name="right_wheel_joint" type="continuous">
@@ -83,5 +89,5 @@
         <collision>
             <geometry>
-                <cylinder length="0.08" radius="0.17" />/>
+                <sphere radius="0.17" />/>
             </geometry>
         </collision>
@@ -90,25 +96,62 @@
         </xacro:inertial_cylinder>
     </link>
-    <!-- CASTER WHEEL -->
-    <joint name="caster_wheel_joint" type="fixed">
-        <parent link="chassis"/>
-        <child link="caster_wheel"/>
-        <origin xyz="0.72 0 0" rpy="0 0 0"/>
+    <gazebo reference="right_wheel">
+        <material>Gazebo/Grey</material>
+    </gazebo>
+    <!--  LEFT FRONT WHEEL LINK  -->
+    <joint name="left_front_wheel_joint" type="fixed">
+        <parent link="base_link"/>
+        <child link="left_front_wheel"/>
+        <origin xyz="0.5 0.285 -0.04" rpy="-${pi/2} 0 0"/>
+        <axis xyz="0 0 2"/>
     </joint>
-    <link name="caster_wheel">
+    <link name="left_front_wheel">
         <visual>
             <geometry>
-                <sphere radius="0.17" />
+                <cylinder length="0.08" radius="0.13" />/>
             </geometry>
-            <material name="black"/>
+            <material name="blue"/>
         </visual>
         <collision>
             <geometry>
-                <sphere radius="0.17" />
+                <sphere radius="0.13" />
             </geometry>
         </collision>
-        <xacro:inertial_sphere mass="1" radius="0.17">
+        <xacro:inertial_cylinder mass="1" length="0.08" radius="0.13">
             <origin xyz="0 0 0" rpy="0 0 0"/>
-        </xacro:inertial_sphere>
-</link>
+        </xacro:inertial_cylinder>
+    </link>
+    <gazebo reference="left_front_wheel">
+        <material>Gazebo/Grey</material>
+        <mu1 value="0.001"/>
+        <mu2 value="0.001"/>
+    </gazebo>
+    <!--  RIGHT FRONT WHEEL LINK  -->
+    <joint name="right_front_wheel_joint" type="fixed">
+        <parent link="base_link"/>
+        <child link="right_front_wheel"/>
+        <origin xyz="0.5 -0.285 -0.04" rpy="${pi/2} 0 0"/>
+        <axis xyz="0 0 -2"/>
+    </joint>
+    <link name="right_front_wheel">
+        <visual>
+            <geometry>
+                <cylinder length="0.08" radius="0.13" />/>
+            </geometry>
+            <material name="blue"/>
+        </visual>
+        <collision>
+            <geometry>
+                <sphere radius="0.13" />
+            </geometry>
+        </collision>
+        <xacro:inertial_cylinder mass="1" length="0.08" radius="0.13">
+            <origin xyz="0 0 0" rpy="0 0 0"/>
+        </xacro:inertial_cylinder>
+    </link>
+    <gazebo reference="right_front_wheel">
+        <material>Gazebo/Grey</material>
+        <mu1 value="0.001"/>
+        <mu2 value="0.001"/>
+    </gazebo>
 </robot>
